File: EPI.kicad_sch (KiCad schematic)
At the start: 5 parts

Commit message: Changed Schematic for changing load resistance rather than input resistance on C1
Parts:
- R1: value R -> 0KR
- R2: value R -> {Range}R
Changed lines of the file:
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@@
 				)
 			)
-			(table_cell "R1"
+			(table_cell "R2\n"
 				(exclude_from_sim no)
 				(at 54.61 53.34 0)
@@
 				)
 			)
-			(table_cell "R2"
+			(table_cell "R1\n"
 				(exclude_from_sim no)
 				(at 54.61 55.88 0)
@@
 				)
 			)
-			(table_cell "1K"
+			(table_cell "0K"
 				(exclude_from_sim no)
 				(at 74.93 55.88 0)
@@
 			)
 		)
-		(property "Value" "R"
+		(property "Value" "0KR"
 			(at 54.61 21.59 90)
 			(show_name no)
@@
 			)
 		)
-		(property "Value" "R"
+		(property "Value" "{Range}R"
 			(at 50.8 35.5599 0)
 			(show_name no)

Commit message: Changed schematic dimensions to better reflect sizing requirements and better fit in external tooling.
Parts:
- R1: value 0KR -> 0R
Changed lines of the file:
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@@
 	(generator "eeschema")
 	(generator_version "10.0")
-	(paper "User" 152.4 190.5)
+	(paper "User" 132.08 152.4)
 	(title_block
 		(title "EPI Circuit Diagram")
@@
 				)
 			)
-			(table_cell "0K"
+			(table_cell "0R\n"
 				(exclude_from_sim no)
 				(at 74.93 55.88 0)
@@
 			)
 		)
-		(property "Value" "0KR"
+		(property "Value" "0R"
 			(at 54.61 21.59 90)
 			(show_name no)
